Commit message: Kinect2 Target don't requite orientation any more

File: boxy_description_urdf/boxy_description.urdf (robot description, URDF)
Before this commit: robot boxy_description, 78 links, 77 joints
Links:
- added link neck_look_target_2
- added link neck_look_target_3
- added link neck_look_target_4
Joints:
- added joint head1: type continuous, parent neck_look_target, child neck_look_target_2, origin xyz=0 0 0 rpy=0 0 0, axis 0 0 1
- added joint head2: type continuous, parent neck_look_target_2, child neck_look_target_3, origin xyz=0 0 0 rpy=0 0 0, axis 0 1 0
- added joint head3: type continuous, parent neck_look_target_3, child neck_look_target_4, origin xyz=0 0 0 rpy=0 0 0, axis 1 0 0

File: boxy_description_urdf/boxy_description.urdf.xacro (robot description, xacro)
@@ -5,14 +5,15 @@
 	<xacro:include filename="$(find iai_wsg_50_description)/urdf/wsg_50.urdf.xacro"/>
 	<xacro:include filename="$(find iai_kms_40_description)/urdf/kms_40.urdf.xacro"/>
-        <include filename="$(find iai_adapters_description)/urdf/lwr4_cabling_adaptor.urdf.xacro" />
+    <xacro:include filename="$(find iai_adapters_description)/urdf/lwr4_cabling_adaptor.urdf.xacro" />
 	<!--xacro:include filename="$(find iai_boxy_description)/sensors/kinect.urdf.xacro"/-->
 	<xacro:include filename="$(find iai_adapters_description)/urdf/adapter_fwa050_wsg50.urdf.xacro"/>
 	<xacro:include filename="$(find iai_adapters_description)/urdf/adapter_kms40_fwk050.urdf.xacro"/>
-        <xacro:include filename="$(find iai_adapters_description)/urdf/fwk_fwa_050.urdf.xacro"/>
+    <xacro:include filename="$(find iai_adapters_description)/urdf/fwk_fwa_050.urdf.xacro"/>
 	<xacro:include filename="$(find iai_adapters_description)/urdf/adapter_boxy_ur3.urdf.xacro"/>
     <xacro:include filename="$(find iai_ur_description)/urdf/ur3.urdf.xacro" />
 	<xacro:include filename="$(find iai_kinect2_description)/urdf/kinect2.urdf.xacro"/>
 	<xacro:include filename="$(find iai_adapter_iso50_kinect2_description)/urdf/adapter_iso50_kinect2.urdf.xacro"/>
-	<xacro:include filename="$(find iai_kinect2_look_target)/urdf/kinect2_target.urdf.xacro"/>
+<!--	<xacro:include filename="$(find iai_kinect2_look_target)/urdf/kinect2_target.urdf.xacro"/> -->
+	<xacro:include filename="$(find boxy_description_urdf)/kinect2_target.urdf.xacro"/>
 	<!-- Property definitions e.g. constants -->
 	<xacro:property name="head_joint_x" value="0.2" />

Commit message: The position of the arms is being tracked

File: boxy_description_urdf/boxy_description.urdf (robot description, URDF)
Before this commit: robot boxy_description, 81 links, 80 joints
Links:
- link neck_look_target: geometry visual cylinder length=0.35 radius=0.035

File: boxy_description_urdf/kinect2_target.urdf.xacro (robot description, xacro)
@@ -20,5 +20,5 @@
 				</geometry>
 				<material name="blue">
-					<color rgba="0 0.1 0.8 1"/>
+					<color rgba="0.2 0.2 0.7 1"/>
 				</material>
 			</visual>
@@ -47,5 +47,5 @@
 		<link name="${prefix}_look_target_4"/>
 	</xacro:macro>
-	<xacro:property name="R" value="0.01" />
-	<xacro:property name="Length" value="0.1" />
+	<xacro:property name="R" value="0.035" />
+	<xacro:property name="Length" value="0.35" />
 </robot>

Commit message: Selecting between different plans before executing.

File: boxy_description_urdf/boxy_description.urdf (robot description, URDF)
Before this commit: robot boxy_description, 81 links, 80 joints
Links:
- added link shoulder_kinect_link; collision sphere radius=0.0005; visual mesh filename=package://iai_kinect_description/meshes/68-04546_Kinect_Sen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 scale=0.001 0.001 0.001
Joints:
- added joint shoulder_kinect_joint: type fixed, parent base_link, child shoulder_kinect_link, origin xyz=-0.00585394 -0.52064754 1.46001 rpy=0.01708077682636155 0.0085798647123734 -0.00929470452726490
- joint triangle_base_joint: origin xyz=0.0786889663592487 0.0986351579738104 0.906352096493862 rpy=4.70695928 6.28217403836 1.56327975371 -> xyz=0.0786889663592487 0.0986351579738104 0.996332096493862 rpy=4.70695928 6.28217403836 1.56327975371

File: boxy_description_urdf/kinect2_target.urdf.xacro (robot description, xacro)
@@ -47,5 +47,5 @@
 		<link name="${prefix}_look_target_4"/>
 	</xacro:macro>
-	<xacro:property name="R" value="0.035" />
+	<xacro:property name="R" value="0.03" />
 	<xacro:property name="Length" value="0.35" />
 </robot>

File: boxy_description_urdf/ur3.urdf.xacro (robot description, xacro)
@@ -80,5 +80,6 @@
       </xacro:unless>
       <xacro:if value="${joint_limited}">
-        <limit lower="${-pi}" upper="${pi}" effort="330.0" velocity="2.16"/>
+        <!--limit lower="${-pi}" upper="${pi}" effort="330.0" velocity="2.16"/-->
+				<limit lower="${-1.5*pi}" upper="${1.5*pi}" effort="330.0" velocity="2.16"/>
       </xacro:if>
       <dynamics damping="0.0" friction="0.0"/>
