Commit message: Adding movement contraints

File: boxy_description_urdf/boxy_description.urdf.xacro (robot description, xacro)
@@ -63,4 +63,24 @@
 			<pose xyz="0 0 0" rpy="0 0 0" />
 		</xacro:kinect2_target_xacro>
+    <!-- Box that limits the position if the head while planning -->
+    <xacro:macro parent="base_link" name="limit_box">
+			<link name="box">
+			  <visual>
+				  <origin rpy="0 0 0" xyz="0.2 0.3 1.2"/>
+					<geometry>
+						<box size="1.05 0.05 0.05"/>
+					</geometry>
+					<material name="box_color">
+						<color rgba="0.2 0.2 0.2 1"/>
+					</material>
+			 	</visual>
+			 	<collision>
+        	<origin rpy="0 0 0" xyz="0.2 0.3 1.2"/>
+        	<geometry>
+         		<box size="1.3 1.3 0.1"/>
+        	</geometry>
+      	</collision>
+		  </link>
+		</xacro:macro>
         <!-- /NEW NECK ASSEMBLY -->
         <!-- OLD NEW ASSEMBLY -->
